File: projects/moloch/moloch.kicad_pcb (KiCad board)
At the start: 2 copper layers, 76 x 34 mm, 11 parts

Commit message: completed rev1
Parts:
- added button: Momentary_Button, gnawman:Momentary_Button, F.Cu at (131.2, 35.5)
- added button: Momentary_Button, gnawman:Momentary_Button, F.Cu at (104.8, 35.5)
- moved button 0.50 mm to (97.8, 75.5)
- moved button 0.50 mm to (130.2, 75.5)
Connections:
- MCU1 pad 1: (no net) -> START
- MCU1 pad 13: (no net) -> SELECT
- MCU1 pad 16: (no net) -> RIGHT
- MCU1 pad 17: (no net) -> DOWN
- MCU1 pad 18: (no net) -> LEFT
- MCU1 pad 19: (no net) -> UP
- MCU1 pad 20: (no net) -> MREC
- MCU1 pad 4: (no net) -> L
- MCU1 pad 5: (no net) -> A
- MCU1 pad 6: (no net) -> B
- MCU1 pad 7: (no net) -> R
- MCU1 pad 8: (no net) -> MPLY
- button pad 1: (no net) -> R
- button pad 1: (no net) -> LEFT
- button pad 1: (no net) -> START
- button pad 1: (no net) -> A
- button pad 1: (no net) -> DOWN
- button pad 1: (no net) -> L
- button pad 1: (no net) -> B
- button pad 1: (no net) -> SELECT
- button pad 1: (no net) -> UP
- button pad 1: (no net) -> RIGHT
Routing:
- net B: track 0.00 -> 38.8 mm
- net LEFT: track 0.00 -> 38.8 mm
- net A: track 0.00 -> 36.4 mm
- net DOWN: track 0.00 -> 36.4 mm
- net UP: track 0.00 -> 33.2 mm
- net R: track 0.00 -> 33.2 mm
- net MREC: track 0.00 -> 21.8 mm
- net MPLY: track 0.00 -> 21.8 mm
- net L: track 0.00 -> 15.7 mm
- net RIGHT: track 0.00 -> 15.7 mm
- net START: track 0.00 -> 12.5 mm
- net SELECT: track 0.00 -> 12.5 mm
Other:
- board text added: "by gnawman"
- board text added: "rev1"
- board text added: "thorny devil"
