File: projects/thorny_devil/thorny_devil.kicad_pcb (KiCad board)
At the start: 2 copper layers, 76 x 34 mm, 13 parts

Commit message: final rev1 commit before manufacture
Parts:
- added ?: , , F.Cu at (94.2, 68.8)
- added ?: , , F.Cu at (92.5, 67.0)
- added ?: , , F.Cu at (88.9, 63.4)
- added ?: , , F.Cu at (141.3, 65.2)
- added ?: , , F.Cu at (143.1, 63.4)
- added ?: , , F.Cu at (90.7, 65.2)
- added ?: , , F.Cu at (137.8, 68.8)
- added ?: , , F.Cu at (139.5, 67.0)
- moved button 1.12 mm to (143.2, 37.5)
- moved button 1.12 mm to (76.5, 49.8)
- moved button 1.12 mm to (155.5, 53.8)
- moved button 1.12 mm to (92.8, 37.5)
- moved button 0.50 mm to (139.2, 66.0)
- moved button 0.50 mm to (88.8, 66.0)
- moved button 0.50 mm to (127.0, 49.8)
- moved button 0.50 mm to (105.0, 53.8)
Connections:
- MCU1 pad 1: START -> RSTICKX
- MCU1 pad 13: SELECT -> RSTICKY
- MCU1 pad 14: (no net) -> LSTICKY
- MCU1 pad 15: (no net) -> RIGHT
- MCU1 pad 16: RIGHT -> LSTICKX
- MCU1 pad 2: (no net) -> START
- MCU1 pad 24: (no net) -> CAPTCH
- MCU1 pad 3: (no net) -> SELECT
- MCU1 pad 9: (no net) -> VCC
Routing:
- net VCC: track 0.00 -> 82.1 mm
- net RSTICKY: track 0.00 -> 34.1 mm
- net RSTICKX: track 0.00 -> 20.5 mm
- net LSTICKX: track 0.00 -> 20.0 mm
- net LSTICKY: track 0.00 -> 18.2 mm
- net SELECT: track 12.5 -> 29.9 mm
- net CAPTCH: track 0.00 -> 9.49 mm, vias 0 -> 1
- net RIGHT: track 15.7 -> 18.2 mm
- net START: track 12.5 -> 13.6 mm
- net B: track 38.8 -> 37.9 mm
- net LEFT: track 38.8 -> 37.9 mm
- net UP: track 33.2 -> 32.6 mm
- net R: track 33.2 -> 32.6 mm
- added copper zone on B.Cu, net CAPTCH
Other:
- outline, holes or cut-outs redrawn
